File: NEW OBC ADCS/OBC/9DOF.kicad_sch (KiCad schematic)
At the start: 6 parts, among them U3 LSM9DS1TR

Commit message: Schematic Finished
Parts:
- C12, C13, C6: footprint Capacitor_SMD:C_0603_1608Metric -> Capacitor_SMD:C_0402_1005Metric; JLCPCB # (none) -> C85953
- C14: footprint Capacitor_SMD:C_0603_1608Metric -> Capacitor_SMD:C_0402_1005Metric; JLCPCB # C2655096 -> C668351
- C5: footprint Capacitor_SMD:C_0603_1608Metric -> Capacitor_SMD:C_0402_1005Metric; JLCPCB # (none) -> C162148
- U3: JLCPCB # (none) -> C2655096
