File: NEW OBC ADCS/OBC/CSS.kicad_sch (KiCad schematic)
At the start: 16 parts, among them J1 Conn_01x04_MountingPin, J7 Conn_01x08_MountingPin, U6 OPA4330, U7 OPA4330

Commit message: Schematic Finished
Parts:
- C26, C31, C32, C33, C34, C35: value 150p -> 220p; footprint Skripsie:C_0201_0603Metric -> Capacitor_SMD:C_0402_1005Metric; JLCPCB # (none) -> C3865471
- R10, R11, R12, R7, R8, R9: value 560 -> 470; footprint Skripsie:R_0201_0603Metric -> Resistor_SMD:R_0402_1005Metric; JLCPCB # (none) -> C491160
- U6, U7: JLCPCB # (none) -> C2059987
Other:
- note added: "Opamps are based on BPW34 photodiodes 50uA @ 1 mW/m^2 Which has a value of 6.9 mA @ 1380W/m^2 VCC of 3.3 V is chosen so: Rf = 3 V / 6.9 mA = 470 ohm 12-bit/16-bit ADCs with maximum voltage of 3,3V Thus resolution is 3.3/(2^12-1)=805.9uV/bit Can be increased ti 3.3/(2^16-1)=50.35uV/bit Thus smallest output current that can be measured is 805.9uV/470ohm = 1.715uA 50.35uV/470ohm = 107.1nA Cf = sqrt(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"
