File: NEW OBC ADCS/OBC/Clocks.kicad_sch (KiCad schematic)
At the start: 6 parts, among them Y3 32.768 kHz, Y4 25 MHz

Commit message: Schematic Finished
Parts:
- C1, C2: value 2p -> 8p; footprint Skripsie:C_0201_0603Metric -> Capacitor_SMD:C_0402_1005Metric; JLCPCB # (none) -> C701199
- C3, C4: value 27p -> 12p; footprint Skripsie:C_0201_0603Metric -> Capacitor_SMD:C_0402_1005Metric; JLCPCB # (none) -> C782159
- Y3: JLCPCB # (none) -> C2449839
- Y4: value 25 MHz -> 80 MHz; JLCPCB # (none) -> C2451101
Other:
- note added: "Cload = (Cl1xCl2)/(Cl1+Cl2)+2pf"
- note removed: "Cload = (Cl1+Cl2)/(Cl1xCl2)+Cs"
