File: NEW OBC ADCS/OBC/DBC.kicad_sch (KiCad schematic)
At the start: 1 part, among them P2 DF40C-50DS-0.4V(51)

Commit message: Schematic Finished
Parts:
- removed P2: DF40C-50DS-0.4V(51), Skripsie:HRS_DF40C-50DS-0.4V(51), symbol DF40C-50DS-0.4V_51_:DF40C-50DS-0.4V(51)
- added J4: Conn_02x10_Counter_Clockwise, Connector_PinHeader_1.27mm:PinHeader_2x10_P1.27mm_Vertical_SMD, symbol Connector_Generic:Conn_02x10_Counter_Clockwise
Connections:
- new net 3v3: J4.2 (Pin_2), J4.9 (Pin_9)
- new net 5V: J4.10 (Pin_10), J4.3 (Pin_3)
- new net ADC: J4.6 (Pin_6)
- new net CAN-CLK: J4.11 (Pin_11)
- new net CAN-DAT: J4.12 (Pin_12)
- new net DAC: J4.5 (Pin_5)
- new net GND: J4.1 (Pin_1), J4.8 (Pin_8)
- new net I2C-SCL: J4.20 (Pin_20)
- new net I2C-SDA: J4.19 (Pin_19)
- new net PPS: J4.4 (Pin_4)
- new net SPI-CLK: J4.14 (Pin_14)
- new net SPI-CS: J4.13 (Pin_13)
- new net SPI-MISO: J4.16 (Pin_16)
- new net SPI-MOSI: J4.15 (Pin_15)
- new net USART-RX: J4.17 (Pin_17)
- new net USART-TX: J4.18 (Pin_18)
- new net VBAT: J4.7 (Pin_7)
- no-connect marks 18 -> 0
Other:
- note added: "Qty | Module | Pins - 1 I2C 2 - 1 USART 2 - 1 ADC 1 - 1 DAC 1 - 1 SPI 4 - 1 CAN 2 - 2 3V 2 - 2 5V 2 - 2 GND 2 - 1 PPS 1 - 1 VBAT 1"
- company: (none) -> 22619291
