File: NEW OBC ADCS/OBC/MSD.kicad_sch (KiCad schematic)
At the start: 8 parts, among them J6 Micro_SD_Card

Commit message: Schematic Finished
Parts:
- C30: footprint Capacitor_SMD:C_0603_1608Metric -> Capacitor_SMD:C_0402_1005Metric; JLCPCB # (none) -> C668351
- J6: footprint DM3CS-SF:HRS_DM3CS-SF -> Skripsie:microSD_HC_Hirose_DM3AT-SF-PEJM5; JLCPCB # (none) -> C114218
- R27, R28, R29, R30, R31, R32: footprint Resistor_SMD:R_0603_1608Metric -> Resistor_SMD:R_0402_1005Metric; JLCPCB # (none) -> C25765
