File: NEW OBC ADCS/OBC/RS485.kicad_sch (KiCad schematic)
At the start: 7 parts, among them U4 MAX485ESA+T

Commit message: Schematic Finished
Parts:
- C8: footprint Capacitor_SMD:C_0603_1608Metric -> Capacitor_SMD:C_0402_1005Metric; JLCPCB # (none) -> C85953
- C9: footprint Capacitor_SMD:C_0603_1608Metric -> Capacitor_SMD:C_0402_1005Metric; JLCPCB # (none) -> C668351
- R13, R14, R15: footprint Resistor_SMD:R_0603_1608Metric -> Resistor_SMD:R_0402_1005Metric; JLCPCB # (none) -> C25765
- R23: footprint Resistor_SMD:R_0603_1608Metric -> Resistor_SMD:R_0402_1005Metric; JLCPCB # (none) -> C423316
- U4: value MAX485ESA+T -> LTC2850HDD#PBF; footprint Package_SO:SOIC-8_3.9x4.9mm_P1.27mm -> Skripsie:DFN-8-1EP_3x3mm_P0.5mm_EP1.65x2.38mm; JLCPCB # C19738 -> C682732
