File: NEW OBC ADCS/OBC/OBC.kicad_pcb (KiCad board)
At the start: 4 copper layers, 42 x 42 mm, 130 parts, among them J1 Conn_01x04_MountingPin, J1 Micro_SD_Card, J2 Conn_01x04, J3 Conn_01x08_MountingPin, J4 Conn_01x04_MountingPin, J5 Conn_02x10_Top_Bottom, J6 Micro_SD_Card, J7 Conn_01x08_MountingPin, J8 Conn_01x05, P1 DF40C-50DS-0.4V(51)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

Commit message: Schematic Finished
Parts:
- removed the H1 at (77.7, 76.4)
- removed the H2 at (77.7, 82.9)
- removed the H3 at (77.7, 89.5)
- removed the H4 at (77.7, 96.0)
- removed the J1 at (98.1, 109.9)
- removed P2: DF40C-50DS-0.4V(51), Skripsie:HRS_DF40C-50DS-0.4V(51)
- removed the R5 at (82.2, 94.2)
- added G*** (x2): LOGO, LOGO, B.Cu at (179.8, 34.1)
- added G***: LOGO, LOGO, B.Cu at (177.8, 31.1)
- added H1: ESL_PQ_MountingHole, ESL_PQ:ESL_PQ_MountingHole, F.Cu at (145.0, 26.5)
- added H1: MountingHole_Pad, MountingHole:MountingHole_2.5mm_Pad, F.Cu at (64.6, 72.6)
- added H2: ESL_PQ_MountingHole, ESL_PQ:ESL_PQ_MountingHole, F.Cu at (181.0, 26.5)
- added H2: MountingHole_Pad, MountingHole:MountingHole_2.5mm_Pad, F.Cu at (64.6, 79.1)
- added H3: MountingHole_Pad, MountingHole:MountingHole_2.5mm_Pad, F.Cu at (64.6, 85.7)
- added H3: ESL_PQ_MountingHole, ESL_PQ:ESL_PQ_MountingHole, F.Cu at (145.0, 62.5)
- added H4: ESL_PQ_MountingHole, ESL_PQ:ESL_PQ_MountingHole, F.Cu at (181.0, 62.5)
- added H4: MountingHole_Pad, MountingHole:MountingHole_2.5mm_Pad, F.Cu at (64.6, 92.2)
- added J1: ESL_PQ_MainHeader, ESL_PQ:ESL_PQ_Main_Header, F.Cu at (163.0, 57.1)
- added J1: Conn_01x04_MountingPin, Skripsie:JST_GH_SM04B-GHS-TB_1x04-1MP_P1.25mm_Horizontal, F.Cu at (104.1, 80.5)
- added J4: Conn_02x10_Counter_Clockwise, Connector_PinHeader_1.27mm:PinHeader_2x10_P1.27mm_Vertical_SMD, F.Cu at (93.7, 104.4)
- added U1: STM32L496R_E-G_Tx, Package_QFP:LQFP-64_10x10mm_P0.5mm, F.Cu at (75.1, 76.5)
- C1, C2: value 2p -> 8p; footprint Skripsie:C_0201_0603Metric -> Capacitor_SMD:C_0402_1005Metric
- C12, C13, C14, C16, C17, C18, C19, C20, C21, C22, C23, C30, C5, C6: footprint Skripsie:C_0201_0603Metric -> Capacitor_SMD:C_0402_1005Metric
- C26, C31, C32, C33, C34, C35: value 150p -> 220p; footprint Skripsie:C_0201_0603Metric -> Capacitor_SMD:C_0402_1005Metric
- C3, C4: value 27p -> 12p; footprint Skripsie:C_0201_0603Metric -> Capacitor_SMD:C_0402_1005Metric
- C8, C9: footprint Capacitor_SMD:C_0603_1608Metric -> Capacitor_SMD:C_0402_1005Metric
- J2: footprint Skripsie:PinHeader_1x04_P1.27mm_Vertical -> Skripsie:JST_GH_SM04B-GHS-TB_1x04-1MP_P1.25mm_Horizontal
- J8: footprint Skripsie:PinHeader_1x05_P1.27mm_Vertical -> Connector_JST:JST_GH_SM05B-GHS-TB_1x05-1MP_P1.25mm_Horizontal
- R1, R2: value R -> 165; footprint Resistor_SMD:R_0603_1608Metric -> Resistor_SMD:R_0402_1005Metric
- R10, R11, R12, R7, R8, R9: value 560 -> 470; footprint Skripsie:R_0201_0603Metric -> Resistor_SMD:R_0402_1005Metric
- R13, R14, R15, R18, R21, R22, R23, R6: footprint Resistor_SMD:R_0603_1608Metric -> Resistor_SMD:R_0402_1005Metric
- R27, R28, R29, R30, R31, R32: footprint Skripsie:R_0201_0603Metric -> Resistor_SMD:R_0402_1005Metric
- U4: value MAX485ESA+T -> LTC2850HDD#PBF; footprint Package_SO:SOIC-8_3.9x4.9mm_P1.27mm -> Skripsie:DFN-8-1EP_3x3mm_P0.5mm_EP1.65x2.38mm
- Y4: value 25 MHz -> 80 MHz
- moved J2 87.5 mm to (83.5, 131.0)
- moved J8 60.1 mm to (115.0, 128.3)
- moved C1 45.9 mm to (186.1, 96.9)
- moved C10 45.9 mm to (185.1, 89.4)
- moved C11 45.9 mm to (184.2, 89.4)
- moved C12 45.9 mm to (185.5, 102.8)
- moved C13 45.9 mm to (185.5, 105.5)
- moved C15 45.9 mm to (191.7, 107.9)
- moved C16 45.9 mm to (196.8, 88.1)
- moved C17 45.9 mm to (193.2, 94.3)
- moved C18 45.9 mm to (193.2, 96.8)
- moved C19 45.9 mm to (196.7, 107.3)
- moved C2 45.9 mm to (183.3, 96.9)
- moved C20 45.9 mm to (208.9, 107.4)
- moved C21 45.9 mm to (212.3, 91.8)
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Connections:
- C12 pad 2: DCap -> +3.3V
- C13 pad 1: DCap -> +3.3V
- C14 pad 1: DCap -> +3.3V
- C30 pad 1: Net-(J6-VSS) -> +3.3V
- J2 pad 1: DCap -> +3.3V
- J6 pad 4: DCap -> +3.3V
- J6 pad 6: Net-(J6-VSS) -> GND
- J8 pad 1: DCap -> +3.3V
- R27 pad 1: DCap -> +3.3V
- R28 pad 1: DCap -> +3.3V
- R29 pad 1: DCap -> +3.3V
- R30 pad 1: DCap -> +3.3V
- R31 pad 1: DCap -> +3.3V
- R32 pad 1: DCap -> +3.3V
- U3 pad 1: DCap -> +3.3V
- U3 pad 22: DCap -> +3.3V
- U3 pad 23: DCap -> +3.3V
- U3 pad 3: DCap -> +3.3V
- U6 pad 4: DCap -> +3.3V
- U7 pad 4: DCap -> +3.3V
Other:
- board size 42 x 42 mm -> 74.6 x 102.9 mm
- board text added: "10"
- board text added: "11"
- board text added: "20"
- board text added: "ESL-PQ Rev 1 OBC"

Commit message: N1
Parts:
- moved J2 66.0 mm to (111.8, 71.3)
- moved J8 65.2 mm to (101.2, 64.7)
Changed lines of the file:
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@@
 	(footprint "Connector_JST:JST_GH_SM05B-GHS-TB_1x05-1MP_P1.25mm_Horizontal"
 		(layer "F.Cu")
-		(at 115 128.35)
+		(at 101.15 64.65)
 		(descr "JST GH series connector, SM05B-GHS-TB (http://www.jst-mfg.com/product/pdf/eng/eGH.pdf), generated with kicad-footprint-generator")
 		(tags "connector JST GH horizontal")
@@
 	(footprint "Skripsie:JST_GH_SM04B-GHS-TB_1x04-1MP_P1.25mm_Horizontal"
 		(layer "F.Cu")
-		(at 83.5 131 180)
+		(at 111.775 71.35 180)
 		(descr "JST GH series connector, SM04B-GHS-TB (http://www.jst-mfg.com/product/pdf/eng/eGH.pdf), generated with kicad-footprint-generator")
 		(tags "connector JST GH top entry")

Commit message: Niel 2
Parts:
- added J3: Conn_01x08_MountingPin, Skripsie:JST_GH_SM08B-GHS-TB_1x08-1MP_P1.25mm_Horizontal, F.Cu at (231.5, 112.0)
- added REF**: JST_GH_SM10B-GHS-TB_1x10-1MP_P1.25mm_Horizontal, Connector_JST:JST_GH_SM10B-GHS-TB_1x10-1MP_P1.25mm_Horizontal, F.Cu at (213.0, 112.5)
- added REF**: JST_GH_SM12B-GHS-TB_1x12-1MP_P1.25mm_Horizontal, Connector_JST:JST_GH_SM12B-GHS-TB_1x12-1MP_P1.25mm_Horizontal, F.Cu at (162.0, 113.0)
- moved J6 91.9 mm to (159.7, 88.2), turned to -90 degrees
- moved R27 88.5 mm to (168.0, 98.0), turned to -90 degrees
- moved R28 86.5 mm to (166.0, 98.0), turned to -90 degrees
- moved R29 84.6 mm to (164.0, 98.0), turned to -90 degrees
- moved R30 82.7 mm to (162.0, 98.0), turned to -90 degrees
- moved R31 80.9 mm to (160.1, 98.0), turned to -90 degrees
- moved R32 79.2 mm to (158.1, 98.0), turned to -90 degrees
- moved C30 77.5 mm to (156.1, 98.0), turned to -90 degrees
