File: NEW OBC ADCS/OBC/OBC.kicad_sch (KiCad schematic)
At the start: 33 parts, among them J2 Conn_01x04, J3 ESL_PQ_MainHeader, J8 Conn_01x05, U1 STM32H723VGT6

Commit message: added mcu
Other:
- added sheet Untitled Sheet (MCU.kicad_sch)

Commit message: Niel 2
Other:
- sheet Untitled Sheet renamed MCU

Commit message: Schematic Finished
Parts:
- removed C24, C25: 100n, Skripsie:C_0201_0603Metric, symbol Device:C
- removed C27, C28: 2.2u, Skripsie:C_0201_0603Metric, symbol Device:C
- removed R16, R17, R19, R20, R5: 4k7, Skripsie:R_0201_0603Metric, symbol Device:R
- removed U1: STM32H723VGT6, Skripsie:LQFP-100_14x14mm_P0.5mm, symbol MCU_ST_STM32H7:STM32H723VGTx
- added C7: 100n, symbol Device:C
- added U1: STM32L496R_E-G_Tx, Package_QFP:LQFP-64_10x10mm_P0.5mm, symbol MCU_ST_STM32L4:STM32L496R_E-G_Tx
- C16: footprint Skripsie:C_0201_0603Metric -> Capacitor_SMD:C_0402_1005Metric; JLCPCB # (none) -> C668351
- C17, C18, C19, C20, C21, C22, C23: footprint Skripsie:C_0201_0603Metric -> Capacitor_SMD:C_0402_1005Metric; JLCPCB # (none) -> C85953
- D1, D2: JLCPCB # (none) -> C138543
- J2: footprint Skripsie:PinHeader_1x04_P1.27mm_Vertical -> Skripsie:JST_GH_SM04B-GHS-TB_1x04-1MP_P1.25mm_Horizontal
- J8: footprint Skripsie:PinHeader_1x05_P1.27mm_Vertical -> Connector_JST:JST_GH_SM05B-GHS-TB_1x05-1MP_P1.25mm_Horizontal
- R1, R2: value R -> 165; footprint Resistor_SMD:R_0603_1608Metric -> Resistor_SMD:R_0402_1005Metric; JLCPCB # (none) -> C226689
- R18, R21, R22, R6: footprint Resistor_SMD:R_0603_1608Metric -> Resistor_SMD:R_0402_1005Metric; now not fitted
Connections:
- net +3.3V: no longer C16.1, C17.1, C18.1, C19.1, C20.1, C21.1, C22.1, C23.1
- net GND: now also C7.2, U1.12 (VSSA), U1.18 (VSS), U1.31 (VSS), U1.47 (VSS), U1.63 (VSS)
- net NRST: now also C7.1, U1.7 (NRST)
- new net DCap: C16.1, C17.1, C18.1, C19.1, C20.1, C21.1, C22.1, C23.1, U1.1 (VBAT), U1.13 (VDDA), U1.19 (VDD), U1.32 (VDD), U1.48 (VDDUSB), U1.64 (VDD)
- no-connect marks 38 -> 3
Other:
- removed sheet MCU
- sheet Daughterboard Connector ports: added 3v3, 5V, ADC, CAN-CLK, CAN-DAT, DAC, GND, I2C-SCL, I2C-SDA, PPS, SPI-CLK, SPI-CS, SPI-MISO, SPI-MOSI, USART-RX, USART-TX, VBAT; removed none
- note added: "LED, Resitor Values"
- moved on the sheet: C16, C17, C18, C19, C20, C21, C22, C23, D1, D2, H1, H2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

Commit message: N2
Connections:
- net DCap is gone; now on net +3.3V: C16.1, C17.1, C18.1, C19.1, C20.1, C21.1, C22.1, C23.1, U1.1 (VBAT), U1.13 (VDDA), U1.19 (VDD), U1.32 (VDD), U1.48 (VDDUSB), U1.64 (VDD)
Other:
- note removed: "LED, Resitor Values"
Changed lines of the file:
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@@
 	)
 	(junction
+		(at 170.18 22.86)
+		(diameter 0)
+		(color 0 0 0 0)
+	)
+	(junction
 		(at 124.46 20.32)
 		(diameter 0)
@@
 		)
 	)
-	(text "LED, Resitor Values\n"
-		(exclude_from_sim no)
-		(at 228.092 103.886 0)
-		(effects
-			(font
-				(size 1.27 1.27)
-			)
-		)
-	)
 	(text "Decoupling Capacitors"
 		(exclude_from_sim no)
@@
 					(unit 1)
 				)
+			)
+		)
+	)
+	(symbol
+		(lib_name "+3.3V_1")
+		(lib_id "power:+3.3V")
+		(at 170.18 22.86 0)
+		(unit 1)
+		(exclude_from_sim no)
+		(in_bom yes)
+		(on_board yes)
+		(dnp no)
+		(property "Reference" "#PWR010"
+			(at 170.18 26.67 0)
+			(effects
+				(font
+					(size 1.27 1.27)
+				)
+				(hide yes)
+			)
+		)
+		(property "Value" "+3.3V"
+			(at 174.498 21.082 0)
+			(effects
+				(font
+					(size 1.27 1.27)
+				)
+			)
+		)
+		(property "Footprint" ""
+			(at 170.18 22.86 0)
+			(effects
+				(font
+					(size 1.27 1.27)
+				)
+				(hide yes)
+			)
+		)
+		(property "Datasheet" ""
+			(at 170.18 22.86 0)
+			(effects
+				(font
+					(size 1.27 1.27)
+				)
+				(hide yes)
+			)
+		)
+		(property "Description" "Power symbol creates a global label with name \"+3.3V\""
+			(at 170.18 22.86 0)
+			(effects
+				(font
+					(size 1.27 1.27)
+				)
+				(hide yes)
+			)
+		)
+		(pin "1"
+		)
+		(instances
+			(project "OBC"
+				(path "/1adcb332-7147-4d8f-ae6d-b23e9f9dd677"
+					(reference "#PWR010")
+					(unit 1)
+				)

Commit message: Niel 2
Parts:
- removed U1: STM32L496R_E-G_Tx, Package_QFP:LQFP-64_10x10mm_P0.5mm, symbol MCU_ST_STM32L4:STM32L496R_E-G_Tx
- added U1: STM32L496VGTxP, Package_QFP:LQFP-100_14x14mm_P0.5mm, symbol MCU_ST_STM32L4:STM32L496VGTxP
- added U2: STM32L476R_C-E-G_Tx, Package_QFP:LQFP-64_10x10mm_P0.5mm, symbol MCU_ST_STM32L4:STM32L476R_C-E-G_Tx
Connections:
- new net: U2.18 (VSS), U2.31 (VSS), U2.47 (VSS), U2.63 (VSS)
- new net: U1.10 (VSS), U1.27 (VSS), U1.49 (VSS), U1.74 (VSS), U1.99 (VSS)
Other:
- note added: "Add Daughter Board Connecter Change Holes to 3mm Accelerometer directly connected to the dac adn dac connected to the rocket STM32L496VTG C717701"
