File: OBC - V10/OBC/DBC.kicad_sch (KiCad schematic)
At the start: 1 part, among them J4 Conn_02x20_Odd_Even

Commit message: PQ V12
Other:
- moved on the sheet: J4
Changed lines of the file:
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@@
 	(hierarchical_label "DB16"
 		(shape input)
-		(at 101.6 109.22 0)
+		(at 148.59 102.87 0)
 		(fields_autoplaced yes)
 		(effects
@@
 	(hierarchical_label "DB10"
 		(shape input)
-		(at 101.6 101.6 0)
+		(at 148.59 95.25 0)
 		(fields_autoplaced yes)
 		(effects
@@
 	(hierarchical_label "DB17"
 		(shape input)
-		(at 88.9 111.76 180)
+		(at 135.89 105.41 180)
 		(fields_autoplaced yes)
 		(effects
@@
 	(hierarchical_label "DB38"
 		(shape input)
-		(at 101.6 137.16 0)
+		(at 148.59 130.81 0)
 		(fields_autoplaced yes)
 		(effects
@@
 	(hierarchical_label "DB7"
 		(shape input)
-		(at 88.9 99.06 180)
+		(at 135.89 92.71 180)
 		(fields_autoplaced yes)
 		(effects
@@
 	(hierarchical_label "DB37"
 		(shape input)
-		(at 88.9 137.16 180)
+		(at 135.89 130.81 180)
 		(fields_autoplaced yes)
 		(effects
@@
 	(hierarchical_label "DB4"
 		(shape input)
-		(at 101.6 93.98 0)
+		(at 148.59 87.63 0)
 		(fields_autoplaced yes)
 		(effects
@@
 	(hierarchical_label "DB27"
 		(shape input)
-		(at 88.9 124.46 180)
+		(at 135.89 118.11 180)
 		(fields_autoplaced yes)
 		(effects
@@
 	(hierarchical_label "DB36"
 		(shape input)
-		(at 101.6 134.62 0)
+		(at 148.59 128.27 0)
 		(fields_autoplaced yes)
 		(effects
@@
 	(hierarchical_label "DB15"
 		(shape input)
-		(at 88.9 109.22 180)
+		(at 135.89 102.87 180)
 		(fields_autoplaced yes)
 		(effects
@@
 	(hierarchical_label "DB30"
 		(shape input)
-		(at 101.6 127 0)
+		(at 148.59 120.65 0)
 		(fields_autoplaced yes)
 		(effects
@@
 	(hierarchical_label "DB33"
 		(shape input)
-		(at 88.9 132.08 180)
+		(at 135.89 125.73 180)
 		(fields_autoplaced yes)
 		(effects
@@
 	(hierarchical_label "DB32"
 		(shape input)
-		(at 101.6 129.54 0)
+		(at 148.59 123.19 0)
 		(fields_autoplaced yes)
 		(effects
@@
 	(hierarchical_label "DB3"
 		(shape input)
-		(at 88.9 93.98 180)
+		(at 135.89 87.63 180)
 		(fields_autoplaced yes)
 		(effects
@@
 	(hierarchical_label "DB13"
 		(shape input)
-		(at 88.9 106.68 180)
+		(at 135.89 100.33 180)
 		(fields_autoplaced yes)
 		(effects
@@
 	(hierarchical_label "DB14"
 		(shape input)
-		(at 101.6 106.68 0)
+		(at 148.59 100.33 0)
 		(fields_autoplaced yes)
 		(effects
@@
 	(hierarchical_label "DB5"
 		(shape input)
-		(at 88.9 96.52 180)
+		(at 135.89 90.17 180)
 		(fields_autoplaced yes)
 		(effects
@@
 	(hierarchical_label "DB9"
 		(shape input)
-		(at 88.9 101.6 180)
+		(at 135.89 95.25 180)
 		(fields_autoplaced yes)
 		(effects
@@
 	(hierarchical_label "DB24"
 		(shape input)
-		(at 101.6 119.38 0)
+		(at 148.59 113.03 0)
 		(fields_autoplaced yes)
 		(effects
@@
 	(hierarchical_label "DB1"
 		(shape input)
-		(at 88.9 91.44 180)
+		(at 135.89 85.09 180)
 		(fields_autoplaced yes)
 		(effects
@@
 	(hierarchical_label "DB25"
 		(shape input)
-		(at 88.9 121.92 180)
+		(at 135.89 115.57 180)
 		(fields_autoplaced yes)
 		(effects
@@
 	(hierarchical_label "DB26"
 		(shape input)
-		(at 101.6 121.92 0)
+		(at 148.59 115.57 0)
 		(fields_autoplaced yes)
 		(effects
@@
 	(hierarchical_label "DB35"
 		(shape input)
-		(at 88.9 134.62 180)
+		(at 135.89 128.27 180)
 		(fields_autoplaced yes)
 		(effects
@@
 	(hierarchical_label "DB40"
 		(shape input)
-		(at 101.6 139.7 0)
+		(at 148.59 133.35 0)
 		(fields_autoplaced yes)
 		(effects
@@
 	(hierarchical_label "DB18"
 		(shape input)
-		(at 101.6 111.76 0)
+		(at 148.59 105.41 0)
 		(fields_autoplaced yes)
 		(effects
@@
 	(hierarchical_label "DB31"
 		(shape input)
-		(at 88.9 129.54 180)
+		(at 135.89 123.19 180)
 		(fields_autoplaced yes)
 		(effects
@@
 	(hierarchical_label "DB28"
 		(shape input)
-		(at 101.6 124.46 0)
+		(at 148.59 118.11 0)
 		(fields_autoplaced yes)
 		(effects
@@
 	(hierarchical_label "DB23"
 		(shape input)
-		(at 88.9 119.38 180)
+		(at 135.89 113.03 180)
 		(fields_autoplaced yes)
 		(effects
@@
 	(hierarchical_label "DB8"
 		(shape input)
-		(at 101.6 99.06 0)
+		(at 148.59 92.71 0)
 		(fields_autoplaced yes)
 		(effects
@@
 	(hierarchical_label "DB6"
 		(shape input)
-		(at 101.6 96.52 0)
+		(at 148.59 90.17 0)
 		(fields_autoplaced yes)
 		(effects
@@
 	(hierarchical_label "DB39"
 		(shape input)
-		(at 88.9 139.7 180)
+		(at 135.89 133.35 180)
 		(fields_autoplaced yes)
 		(effects
@@
 	(hierarchical_label "DB19"
 		(shape input)
-		(at 88.9 114.3 180)
+		(at 135.89 107.95 180)
 		(fields_autoplaced yes)
 		(effects
@@
 	(hierarchical_label "DB2"
 		(shape input)
-		(at 101.6 91.44 0)
+		(at 148.59 85.09 0)
 		(fields_autoplaced yes)
 		(effects
@@
 	(hierarchical_label "DB21"
 		(shape input)
-		(at 88.9 116.84 180)
+		(at 135.89 110.49 180)
 		(fields_autoplaced yes)
 		(effects
@@
 	(hierarchical_label "DB12"
 		(shape input)
-		(at 101.6 104.14 0)
+		(at 148.59 97.79 0)
 		(fields_autoplaced yes)
 		(effects
@@
 	(hierarchical_label "DB22"
 		(shape input)
-		(at 101.6 116.84 0)
+		(at 148.59 110.49 0)
 		(fields_autoplaced yes)
 		(effects
@@
 	(hierarchical_label "DB29"
 		(shape input)
-		(at 88.9 127 180)
+		(at 135.89 120.65 180)
 		(fields_autoplaced yes)
 		(effects
@@
 	(hierarchical_label "DB11"
 		(shape input)
-		(at 88.9 104.14 180)
+		(at 135.89 97.79 180)
 		(fields_autoplaced yes)
 		(effects
@@
 	(hierarchical_label "DB34"
 		(shape input)
-		(at 101.6 132.08 0)
+		(at 148.59 125.73 0)
 		(fields_autoplaced yes)
 		(effects
@@
 	(hierarchical_label "DB20"
 		(shape input)
-		(at 101.6 114.3 0)
+		(at 148.59 107.95 0)
 		(fields_autoplaced yes)
 		(effects
@@
 	(symbol
 		(lib_id "Connector_Generic:Conn_02x20_Odd_Even")
-		(at 93.98 114.3 0)
+		(at 140.97 107.95 0)
 		(unit 1)
 		(exclude_from_sim no)
@@
 		(fields_autoplaced yes)
 		(property "Reference" "J4"
-			(at 95.25 85.09 0)
+			(at 142.24 78.74 0)
 			(effects
 				(font
@@
 		)
 		(property "Value" "Conn_02x20_Odd_Even"
-			(at 95.25 87.63 0)
+			(at 142.24 81.28 0)
 			(effects
 				(font
@@
 		)
 		(property "Footprint" "Skripsie:HRS_DF40C-50DS-0.4V(51)"
-			(at 93.98 114.3 0)
+			(at 140.97 107.95 0)
 			(effects
 				(font
@@
 		)
 		(property "Datasheet" "~"
-			(at 93.98 114.3 0)
+			(at 140.97 107.95 0)
 			(effects
 				(font
@@
 		)
 		(property "Description" "Generic connector, double row, 02x20, odd/even pin numbering scheme (row 1 odd numbers, row 2 even numbers), script generated (kicad-library-utils/schlib/autogen/connector/)"
-			(at 93.98 114.3 0)
-			(effects
-				(font
+			(at 140.97 107.95 0)
+			(effects
+				(font
+					(size 1.27 1.27)
+				)
+				(hide yes)
+			)
+		)
+		(property "JLCPCB #" "~"
+			(at 140.97 107.95 0)
+			(effects
+				(font
