File: OBC - V10/OBC/OBC.kicad_sch (KiCad schematic)
At the start: 32 parts, among them J1 Conn_01x05, J2 Conn_01x04, J3 ESL_PQ_MainHeader, U1 STM32L496VGTxP

Commit message: PQ V12
Parts:
- removed U1: STM32L496VGTxP, Package_QFP:LQFP-100_14x14mm_P0.5mm, symbol MCU_ST_STM32L4:STM32L496VGTxP
- added C21: 1u, Skripsie:C_0201_0603Metric, symbol Device:C
- added U1: STM32L496VGTx, Package_QFP:LQFP-100_14x14mm_P0.5mm, symbol MCU_ST_STM32L4:STM32L496VGTx
- C17: renamed from C20; footprint Capacitor_SMD:C_0603_1608Metric -> Skripsie:C_0201_0603Metric
- C20: renamed from C23; value 100n -> 1u
- R15: renamed from R3; now not fitted
- R17: renamed from R5; now not fitted
- R20: renamed from R16; value R -> 4k7; JLCPCB # (none) -> C25765
- R21: renamed from R17; value R -> 4k7; JLCPCB # (none) -> C25765
- R22: renamed from R19; value R -> 4k7; JLCPCB # (none) -> C25765
- R23: renamed from R20; value R -> 4k7; JLCPCB # (none) -> C25765
- renumbered C16 to C13, C17 to C14, C18 to C15, C19 to C16, C21 to C18, C22 to C19, C7 to C22, R6 to R11, R18 to R12, R21 to R13, R22 to R14, R4 to R16, R1 to R18, R2 to R19
Connections:
- net +3.3V: now also C21.1, U1.100 (VDD), U1.11 (VDD), U1.21 (VREF+), U1.22 (VDDA), U1.28 (VDD), U1.50 (VDD), U1.6 (VBAT), U1.73 (VDDUSB), U1.75 (VDD)
- net CSAG: now also U1.3 (PE4)
- net CSM: now also U1.2 (PE3)
- net GND: now also C22.1, C21.2, U1.10 (VSS), U1.19 (VSSA), U1.20 (VREF-), U1.27 (VSS), U1.49 (VSS), U1.74 (VSS), U1.99 (VSS); no longer C22.2
- net I2C-SCL: now also U1.15 (PC0), U1.60 (PD13)
- net I2C-SDA: now also U1.16 (PC1), U1.59 (PD12)
- net NRST: now also C22.2, U1.14 (NRST); no longer C22.1
- net OSC32_IN: now also U1.8 (PC14)
- net OSC32_OUT: now also U1.9 (PC15)
- net OSC_IN: now also U1.12 (PH0)
- net OSC_OUT: now also U1.13 (PH1)
- net RS-EN: now also U1.71 (PA12)
- net SAOG: now also U1.5 (PE6)
- net SAOM: now also U1.4 (PE5)
- net SCL: now also U1.95 (PB8)
- net SDA: now also U1.96 (PB9)
- net SPI MISO: now also U1.52 (PB13)
- net SPI MOSI: now also U1.51 (PB12)
- net SPI NSS: now also U1.54 (PB15)
- net SPI SCK: now also U1.53 (PB14)
- net SWCLK: now also U1.76 (PA14)
- net SWDIO: now also U1.72 (PA13)
- net EPS_RST renamed EPS-RST
- new net DB: U1.17 (PC2), U1.18 (PC3), U1.23 (PA0), U1.24 (PA1), U1.25 (PA2), U1.26 (PA3), U1.31 (PA6), U1.32 (PA7), U1.33 (PC4), U1.34 (PC5), U1.35 (PB0), U1.36 (PB1), U1.43 (PE12), U1.44 (PE13), U1.45 (PE14), U1.46 (PE15), U1.47 (PB10), U1.48 (PB11), U1.55 (PD8), U1.56 (PD9), U1.77 (PA15), U1.78 (PC10), U1.79 (PC11), U1.80 (PC12), U1.81 (PD0), U1.82 (PD1), U1.83 (PD2), U1.86 (PD5), U1.87 (PD6), U1.89 (PB3), U1.90 (PB4), U1.91 (PB5)
- no-connect marks 2 -> 27
Other:
- note added: "Accelerometer directly connected to the dac adn dac connected to the rocket STM32L496VTG C717701"
- note added: "Debug LEDs"
- note removed: "Add Daughter Board Connecter Change Holes to 3mm Accelerometer directly connected to the dac adn dac connected to the rocket STM32L496VTG C717701"
- note removed: "LED"
- note removed: "Make this 0201s"
- moved on the sheet: C13, C14, C15, C16, C17, C18, C19, C20, C22, D1, D2, H1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
