File: OBC - V10/OBC/RS485.kicad_sch (KiCad schematic)
At the start: 7 parts, among them U4 LTC2850HDD#PBF

Commit message: PQ V12
Parts:
- U3: renamed from U4; value LTC2850HDD#PBF -> MAX485EDA; JLCPCB # C682732 -> C19738
- renumbered C8 to C11, C9 to C12, R23 to R10, R13 to R7, R14 to R8, R15 to R9
Changed lines of the file:
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@@
 		(on_board yes)
 		(dnp no)
-		(property "Reference" "U4"
+		(property "Reference" "U3"
 			(at 158.4041 93.98 0)
 			(effects
@@
 			)
 		)
-		(property "Value" "LTC2850HDD#PBF"
+		(property "Value" "MAX485EDA"
 			(at 158.4041 96.52 0)
 			(effects
@@
 			)
 		)
-		(property "Description" "transceiver 2.5Mbps 1/1 SOIC-8 RS-485/RS-422 ICs ROHS"
+		(property "Description" ""
 			(at 165.862 135.382 0)
 			(effects
@@
 			)
 		)
-		(property "JLCPCB #" "C682732"
+		(property "JLCPCB #" "C19738"
 			(at 156.21 110.49 0)
 			(effects
@@
 			(project "OBC"
 				(path "/1adcb332-7147-4d8f-ae6d-b23e9f9dd677/3ee593e4-95d4-4cb2-ba50-581433cc554f"
-					(reference "U4")
+					(reference "U3")
 					(unit 1)
 				)
@@
 		(dnp no)
 		(fields_autoplaced yes)
-		(property "Reference" "R13"
+		(property "Reference" "R7"
 			(at 132.08 119.3799 0)
 			(effects
@@
 			(project "OBC"
 				(path "/1adcb332-7147-4d8f-ae6d-b23e9f9dd677/3ee593e4-95d4-4cb2-ba50-581433cc554f"
-					(reference "R13")
+					(reference "R7")
 					(unit 1)
 				)
@@
 		(on_board yes)
 		(dnp no)
-		(property "Reference" "C8"
+		(property "Reference" "C11"
 			(at 135.89 88.9 0)
 			(effects
@@
 			(project "OBC"
 				(path "/1adcb332-7147-4d8f-ae6d-b23e9f9dd677/3ee593e4-95d4-4cb2-ba50-581433cc554f"
-					(reference "C8")
+					(reference "C11")
 					(unit 1)
 				)
@@
 		(dnp yes)
 		(fields_autoplaced yes)
-		(property "Reference" "R15"
+		(property "Reference" "R9"
 			(at 176.53 119.3799 0)
 			(effects
@@
 			(project "OBC"
 				(path "/1adcb332-7147-4d8f-ae6d-b23e9f9dd677/3ee593e4-95d4-4cb2-ba50-581433cc554f"
-					(reference "R15")
+					(reference "R9")
 					(unit 1)
 				)
@@
 		(dnp no)
 		(fields_autoplaced yes)
-		(property "Reference" "C9"
+		(property "Reference" "C12"
 			(at 147.32 88.8999 0)
 			(effects
@@
 			(project "OBC"
 				(path "/1adcb332-7147-4d8f-ae6d-b23e9f9dd677/3ee593e4-95d4-4cb2-ba50-581433cc554f"
-					(reference "C9")
+					(reference "C12")
 					(unit 1)
 				)
@@
 		(dnp yes)
 		(fields_autoplaced yes)
-		(property "Reference" "R14"
+		(property "Reference" "R8"
 			(at 176.53 88.8999 0)
 			(effects
@@
 			(project "OBC"
 				(path "/1adcb332-7147-4d8f-ae6d-b23e9f9dd677/3ee593e4-95d4-4cb2-ba50-581433cc554f"
-					(reference "R14")
+					(reference "R8")
 					(unit 1)
 				)
@@
 		(dnp no)
 		(fields_autoplaced yes)
-		(property "Reference" "R23"
+		(property "Reference" "R10"
 			(at 180.34 104.1399 0)
 			(effects
@@
 			(project "OBC"
 				(path "/1adcb332-7147-4d8f-ae6d-b23e9f9dd677/3ee593e4-95d4-4cb2-ba50-581433cc554f"
-					(reference "R23")
+					(reference "R10")
 					(unit 1)
 				)
