File: OBC - V12/OBC/OBC.kicad_pcb (KiCad board)
At the start: 4 copper layers, 42 x 42 mm, 64 parts, among them J1 Conn_01x05, J2 Conn_01x04, J3 ESL_PQ_MainHeader, J4 Conn_02x20_Odd_Even, J5 Micro_SD_Card, U1 STM32L496VGTx, U2 LSM9DS1TR, U3 MAX485EDA, Y1 32.768 kHz, Y2 16 MHz

Commit message: FINAL
Parts:
- removed R15, R16, R17: 0, Skripsie:R_0201_0603Metric
- D1, D2, R18, R19: moved to F.Cu
- J2: value Conn_01x04 -> Conn_01x05; footprint Skripsie:PinHeader_1x04_P1.27mm_Vertical -> Skripsie:PinHeader_1x05_P1.27mm_Vertical
- J4: value Conn_02x20_Odd_Even -> Conn_02x25_Odd_Even
- moved G*** 44.5 mm to (250.2, 62.5) (x2)
- moved G*** 44.5 mm to (254.9, 62.5)
- moved R18 21.9 mm to (234.5, 39.5), turned to 90 degrees
- moved D1 20.7 mm to (234.5, 42.8), turned to 90 degrees
- moved R19 17.9 mm to (231.4, 39.5), turned to 90 degrees
- moved D2 16.6 mm to (231.4, 42.8), turned to 90 degrees
- moved J2 2.25 mm to (266.9, 52.0)
- moved C22 2.05 mm to (234.3, 56.8)
- moved J1 2.00 mm to (232.1, 52.0)
- moved C21 1.34 mm to (258.7, 38.2), turned to -90 degrees
- moved C20 0.92 mm to (259.6, 38.2), turned to -90 degrees
- moved U3 0.10 mm to (264.5, 48.1)
Connections:
- net /Daughterboard Connector/DB10 renamed DB10
- net /Daughterboard Connector/DB14 renamed DB14
- net /Daughterboard Connector/DB18 renamed DB18
- net /Daughterboard Connector/DB22 renamed DB22
- net /Daughterboard Connector/DB26 renamed DB26
- net /Daughterboard Connector/DB27 renamed DB27
- net /Daughterboard Connector/DB31 renamed DB31
- net /Daughterboard Connector/DB35 renamed DB35
- net /Daughterboard Connector/DB36 renamed DB36
- net /Daughterboard Connector/DB39 renamed DB39
- net /Daughterboard Connector/DB40 renamed DB40
- net /Daughterboard Connector/DB6 renamed DB6
- J3 pad 6: S1_3V3 -> DCap
- J4 pad 1: /Daughterboard Connector/DB1 -> DB1
- J4 pad 11: /Daughterboard Connector/DB11 -> DB11
- J4 pad 12: /Daughterboard Connector/DB12 -> DB12
- J4 pad 13: /Daughterboard Connector/DB13 -> DB13
- J4 pad 15: /Daughterboard Connector/DB15 -> DB15
- J4 pad 16: /Daughterboard Connector/DB16 -> DB16
- J4 pad 17: /Daughterboard Connector/DB17 -> DB17
- J4 pad 19: /Daughterboard Connector/DB19 -> DB19
- J4 pad 2: /Daughterboard Connector/DB2 -> DB2
- J4 pad 20: /Daughterboard Connector/DB20 -> DB20
- J4 pad 21: /Daughterboard Connector/DB21 -> DB21
- J4 pad 23: /Daughterboard Connector/DB23 -> DB23
- J4 pad 24: /Daughterboard Connector/DB24 -> DB24
- J4 pad 25: /Daughterboard Connector/DB25 -> DB25
- J4 pad 28: /Daughterboard Connector/DB28 -> DB28
- J4 pad 29: /Daughterboard Connector/DB29 -> DB29
- J4 pad 3: /Daughterboard Connector/DB3 -> DB3
- J4 pad 30: /Daughterboard Connector/DB30 -> DB30
- J4 pad 32: /Daughterboard Connector/DB32 -> DB32
- J4 pad 33: /Daughterboard Connector/DB33 -> DB33
- J4 pad 34: /Daughterboard Connector/DB34 -> DB34
- J4 pad 37: /Daughterboard Connector/DB37 -> DB37
- J4 pad 38: /Daughterboard Connector/DB38 -> DB38
- J4 pad 4: /Daughterboard Connector/DB4 -> DB4
- J4 pad 41: (no net) -> DB41
- J4 pad 42: (no net) -> DB42
- J4 pad 43: (no net) -> DB43
- J4 pad 44: (no net) -> DB44
- J4 pad 45: (no net) -> DB45
- J4 pad 46: (no net) -> DB46
- J4 pad 47: (no net) -> DB47
- J4 pad 48: (no net) -> DB48
- J4 pad 49: (no net) -> DB49
- J4 pad 5: /Daughterboard Connector/DB5 -> DB5
- J4 pad 50: (no net) -> DB50
- J4 pad 7: /Daughterboard Connector/DB7 -> DB7
- J4 pad 8: /Daughterboard Connector/DB8 -> DB8
- J4 pad 9: /Daughterboard Connector/DB9 -> DB9
- U1 pad 17: DB -> DB30
- U1 pad 18: DB -> DB34
- U1 pad 23: DB -> DB32
- U1 pad 24: DB -> DB28
- U1 pad 25: DB -> DB38
- U1 pad 26: DB -> DB42
- U1 pad 29: unconnected-(U1-PA4-Pad29) -> DB46
- U1 pad 30: unconnected-(U1-PA5-Pad30) -> DB50
- U1 pad 31: DB -> DB49
- U1 pad 32: DB -> DB45
- U1 pad 33: DB -> DB41
- U1 pad 34: DB -> DB37
- U1 pad 35: DB -> DB33
- U1 pad 36: DB -> DB29
- U1 pad 43: DB -> DB25
- U1 pad 44: DB -> DB21
- U1 pad 45: DB -> DB17
- U1 pad 46: DB -> DB13
- U1 pad 47: DB -> DB9
- U1 pad 48: DB -> DB5
- U1 pad 55: DB -> DB20
- U1 pad 56: DB -> DB24
- U1 pad 57: unconnected-(U1-PD10-Pad57) -> TX
- U1 pad 58: unconnected-(U1-PD11-Pad58) -> PWR
- U1 pad 68: unconnected-(U1-PA9-Pad68) -> USART TX
- U1 pad 69: unconnected-(U1-PA10-Pad69) -> USART RX
- U1 pad 70: unconnected-(U1-PA11-Pad70) -> PPS
- U1 pad 77: DB -> DB2
- U1 pad 78: DB -> DB1
- U1 pad 79: DB -> DB16
- U1 pad 80: DB -> DB12
- U1 pad 81: DB -> DB8
- U1 pad 82: DB -> DB4
- U1 pad 83: DB -> DB3
- U1 pad 86: DB -> DB7
- U1 pad 87: DB -> DB11
- U1 pad 89: DB -> DB15
- U1 pad 90: DB -> DB19
- U1 pad 91: DB -> DB23
- U1 pad 97: unconnected-(U1-PE0-Pad97) -> EPS-RST
Routing:
- net NRST: track 2.18 -> 62.9 mm, vias 0 -> 2
- net I2C-SDA: track 2.50 -> 62.1 mm, vias 0 -> 2
- net I2C-SCL: track 2.44 -> 56.8 mm, vias 0 -> 2
- net /Daughterboard Connector/DB8: track 44.3 -> 0.00 mm, vias 4 -> 0
- net /Daughterboard Connector/DB4: track 37.2 -> 0.00 mm, vias 4 -> 0
- net DB16: track 0.00 -> 34.4 mm, vias 0 -> 2
- net DB12: track 0.00 -> 32.7 mm, vias 0 -> 2
- net /Daughterboard Connector/DB16: track 32.3 -> 0.00 mm, vias 1 -> 0
- net DB8: track 0.00 -> 31.8 mm, vias 0 -> 2
- net /Daughterboard Connector/DB12: track 31.1 -> 0.00 mm, vias 1 -> 0
- net DB27: track 41.7 -> 11.2 mm, vias 2 -> 1
- net DB35: track 40.0 -> 10.2 mm, vias 2 -> 1
- net DB31: track 40.5 -> 10.9 mm, vias 2 -> 1
- net DB23: track 0.00 -> 28.9 mm, vias 0 -> 2
- net DB2: track 0.00 -> 28.6 mm, vias 0 -> 2
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Other:
- outline, holes or cut-outs redrawn
- board text added: "D.P. Theron C. Flood"
