File: OBC - V12/OBC/OBC.kicad_sch (KiCad schematic)
At the start: 33 parts, among them J1 Conn_01x05, J2 Conn_01x04, J3 ESL_PQ_MainHeader, U1 STM32L496VGTx

Commit message: FINAL
Parts:
- removed J2: Conn_01x04, Skripsie:PinHeader_1x04_P1.27mm_Vertical, symbol Connector_Generic:Conn_01x04
- removed R15, R16, R17: 0, Skripsie:R_0201_0603Metric, symbol Device:R
- added J2: Conn_01x05, Skripsie:PinHeader_1x05_P1.27mm_Vertical, symbol Connector_Generic:Conn_01x05
Connections:
- net S1_3V3 is gone; now on net +3.3V: J3.6 (Pin_6)
- net +3.3V: now also J2.1 (Pin_1)
- net EPS-RST: now also U1.97 (PE0)
- net GND: now also J2.2 (Pin_2)
- net PPS: now also U1.70 (PA11)
- net PWR: now also U1.58 (PD11)
- net TX: now also U1.57 (PD10)
- net USART RX: now also U1.69 (PA10), J2.4 (Pin_4)
- net USART TX: now also U1.68 (PA9), J2.3 (Pin_3)
- net DB46: now reaches U1.29 (PA4)
- net DB50: now reaches U1.30 (PA5)
- removed net DB: U1.17 (PC2), U1.18 (PC3), U1.23 (PA0), U1.24 (PA1), U1.25 (PA2), U1.26 (PA3), U1.31 (PA6), U1.32 (PA7), U1.33 (PC4), U1.34 (PC5), U1.35 (PB0), U1.36 (PB1), U1.43 (PE12), U1.44 (PE13), U1.45 (PE14), U1.46 (PE15), U1.47 (PB10), U1.48 (PB11), U1.55 (PD8), U1.56 (PD9), U1.77 (PA15), U1.78 (PC10), U1.79 (PC11), U1.80 (PC12), U1.81 (PD0), U1.82 (PD1), U1.83 (PD2), U1.86 (PD5), U1.87 (PD6), U1.89 (PB3), U1.90 (PB4), U1.91 (PB5)
- new net DB1: U1.78 (PC10)
- new net DB11: U1.87 (PD6)
- new net DB12: U1.80 (PC12)
- new net DB13: U1.46 (PE15)
- new net DB15: U1.89 (PB3)
- new net DB16: U1.79 (PC11)
- new net DB17: U1.45 (PE14)
- new net DB19: U1.90 (PB4)
- new net DB2: U1.77 (PA15)
- new net DB20: U1.55 (PD8)
- new net DB21: U1.44 (PE13)
- new net DB23: U1.91 (PB5)
- new net DB24: U1.56 (PD9)
- new net DB25: U1.43 (PE12)
- new net DB28: U1.24 (PA1)
- new net DB29: U1.36 (PB1)
- new net DB3: U1.83 (PD2)
- new net DB30: U1.17 (PC2)
- new net DB32: U1.23 (PA0)
- new net DB33: U1.35 (PB0)
- new net DB34: U1.18 (PC3)
- new net DB37: U1.34 (PC5)
- new net DB38: U1.25 (PA2)
- new net DB4: U1.82 (PD1)
- new net DB41: U1.33 (PC4)
- new net DB42: U1.26 (PA3)
- new net DB45: U1.32 (PA7)
- new net DB49: U1.31 (PA6)
- new net DB5: U1.48 (PB11)
- new net DB7: U1.86 (PD5)
- new net DB8: U1.81 (PD0)
- new net DB9: U1.47 (PB10)
- no-connect marks 27 -> 23
Other:
- sheet Daughterboard Connector ports: added DB41, DB42, DB43, DB44, DB45, DB46, DB47, DB48, DB49, DB50; removed none
- note removed: "Power Selection"
- moved on the sheet: R20, R21
